Commit message: use rtk data

File: launch/include/config/robot.urdf.xacro (robot description, xacro)
@@ -27,3 +27,16 @@
     <origin xyz="0 0 0" rpy="0 0 0" />
   </joint>
+  <link name="gnss_link"> </link>
+  <joint name="gnss_joint" type="fixed">
+    <parent link="chassis_link" />
+    <child link="gnss_link" />
+    <origin xyz="0 0 0" rpy="0 0 0" />
+  </joint>
+  <!-- 添加自己的传感器坐标系到base_link变换关系 -->
+  <link name="/imu"> </link>
+  <joint name="/imu_joint" type="fixed">
+    <parent link="chassis_link" />
+    <child link="/imu" />
+    <origin xyz="0 0 0" rpy="0 0 0" />
+  </joint>
 </robot>
